Commit message: Add gazebo_walker.launch.py: spawn + bridge the legged walker, drive it via champ_base
Spawns cavex_walker in the dry-cave section, bridges its sensors (lidar,
camera, IMU, clock) and ground-truth pose over gz-transport, and launches
champ_base's quadruped_controller_node so /cmd_vel actually drives leg
trajectories (the plan's 4 steps covered spawning/bridging but not gait
control, without which the robot could never walk).

- cavex_walker.urdf.xacro: adds the <ros2_control> hardware-interface block
  gz_ros2_control needs (missing entirely before this task -- confirmed by
  a real crash: "no 'ros2_control' tag found in the URDF"), a
  PosePublisher plugin for ground-truth world pose, and a fixed
  <leg>_foot_link per leg so champ's links_map has the real 4-link chain
  its own FK requires (champ/include/champ/quadruped_base/quadruped_leg.h).
- cavex_walker_joints_map.yaml (new): links_map/joints_map for
  quadruped_controller_node, schema read directly from
  champ/include/champ/utils/urdf_loader.h since no example ships anywhere
  in the vendored champ/champ_base source.
- gazebo_walker.launch.py (new): gz_sim + robot_state_publisher + spawn +
  parameter_bridge (lidar topic fixed to the real gz-transport name,
  .../points/points, found via `gz topic -i` per this session's established
  gz-sim topic-naming gotcha) + quadruped_controller_node (cmd_vel/smooth
  remapped to /cmd_vel) + controller_manager spawners for
  joint_state_broadcaster/joint_group_position_controller (empirically
  required -- gz_ros2_control does not auto-activate them).

Verified empirically: full stack launched cleanly, all producer topics
carry real data (lidar/points, camera, imu, model pose matching spawn
location), and publishing to /cmd_vel produces real, changing
joint_trajectory commands in a diagonal-trot pattern.

Co-Authored-By: Claude Sonnet 5 <noreply@anthropic.com>

File: ros2_ws/src/cavex_slam_nav/urdf/cavex_walker.urdf.xacro (robot description, xacro)
@@ -30,6 +30,16 @@
     knee_joint  = CHAMP's "knee"  (pitch, bends the shank)
   CHAMP's config additionally carries a 4th, non-actuated "foot" frame per
-  leg for FK bookkeeping; this file omits it since it isn't a controlled
-  joint and isn't required for gz_ros2_control's command interface.
+  leg for FK bookkeeping; this file omits it as a controlled joint (not
+  needed for gz_ros2_control's command interface) but Task 5 adds a fixed
+  <leg>_foot_link/<leg>_foot_joint pair per leg below anyway: champ's
+  links_map schema (champ/include/champ/utils/urdf_loader.h,
+  champ/include/champ/quadruped_base/quadruped_leg.h's 4-element
+  joint_chain) requires exactly 4 link names per leg to walk the kinematic
+  chain for its own internal forward kinematics (hip -> upper_leg ->
+  lower_leg -> foot). Without a real foot_link offset by -shank_length from
+  knee_link, champ's link chain would be one segment short and its leg IK
+  would be computed for the wrong leg length. See
+  cavex_walker_joints_map.yaml for how links_map/joints_map reference these
+  names.
 -->
 <robot name="cavex_walker" xmlns:xacro="http://ros.org/wiki/xacro">
@@ -134,4 +144,15 @@
       <limit lower="-2.5" upper="0.0" effort="20" velocity="10"/>
     </joint>
+    <!-- Virtual foot frame: fixed, offset by -shank_length from the knee.
+         Not a controlled joint (see header comment) - exists solely so
+         champ's links_map has a real 4th link per leg with the correct
+         shank length baked into its FK, matching quadruped_leg.h's
+         hip/upper_leg/lower_leg/foot 4-element joint_chain. -->
+    <link name="${prefix}_foot_link"/>
+    <joint name="${prefix}_foot_joint" type="fixed">
+      <parent link="${prefix}_knee_link"/>
+      <child link="${prefix}_foot_link"/>
+      <origin xyz="0 0 -${shank_length}" rpy="0 0 0"/>
+    </joint>
   </xacro:macro>
   <xacro:champ_leg prefix="lf" x_sign="1"  y_sign="1"/>
@@ -139,4 +160,44 @@
   <xacro:champ_leg prefix="lh" x_sign="-1" y_sign="1"/>
   <xacro:champ_leg prefix="rh" x_sign="-1" y_sign="-1"/>
+  <!-- ros2_control hardware interface block. Found missing empirically:
+       `gz_ros2_control::GazeboSimROS2ControlPlugin` (the <gazebo><plugin>
+       block above) only supplies the controller_manager YAML - it still
+       needs this separate <ros2_control> tag in the URDF itself to know
+       which joints exist and what command/state interfaces they expose.
+       Without it, gz-sim's controller_manager aborts on spawn with
+       "no 'ros2_control' tag found in the URDF" (std::terminate, process
+       exit 134) - reproduced and confirmed via a real launch attempt
+       before adding this block, not assumed. Hardware plugin name/type
+       confirmed installed, not guessed:
+       `cat /opt/ros/jazzy/share/gz_ros2_control/gz_hardware_plugins.xml`
+       -> pluginlib class name "gz_ros2_control/GazeboSimSystem". Command
+       interface limits match each joint's own <limit> above. -->
+  <xacro:macro name="champ_ros2_control_joint" params="name lower upper">
+    <joint name="${name}">
+      <command_interface name="position">
+        <param name="min">${lower}</param>
+        <param name="max">${upper}</param>
+      </command_interface>
+      <state_interface name="position"/>
+      <state_interface name="velocity"/>
+    </joint>
+  </xacro:macro>
+  <ros2_control name="GazeboSimSystem" type="system">
+    <hardware>
+      <plugin>gz_ros2_control/GazeboSimSystem</plugin>
+    </hardware>
+    <xacro:champ_ros2_control_joint name="lf_hip_joint"   lower="-0.75" upper="0.75"/>
+    <xacro:champ_ros2_control_joint name="lf_thigh_joint" lower="-1.5"  upper="1.5"/>
+    <xacro:champ_ros2_control_joint name="lf_knee_joint"  lower="-2.5"  upper="0.0"/>
+    <xacro:champ_ros2_control_joint name="rf_hip_joint"   lower="-0.75" upper="0.75"/>
+    <xacro:champ_ros2_control_joint name="rf_thigh_joint" lower="-1.5"  upper="1.5"/>
+    <xacro:champ_ros2_control_joint name="rf_knee_joint"  lower="-2.5"  upper="0.0"/>
+    <xacro:champ_ros2_control_joint name="lh_hip_joint"   lower="-0.75" upper="0.75"/>
+    <xacro:champ_ros2_control_joint name="lh_thigh_joint" lower="-1.5"  upper="1.5"/>
+    <xacro:champ_ros2_control_joint name="lh_knee_joint"  lower="-2.5"  upper="0.0"/>
+    <xacro:champ_ros2_control_joint name="rh_hip_joint"   lower="-0.75" upper="0.75"/>
+    <xacro:champ_ros2_control_joint name="rh_thigh_joint" lower="-1.5"  upper="1.5"/>
+    <xacro:champ_ros2_control_joint name="rh_knee_joint"  lower="-2.5"  upper="0.0"/>
+  </ros2_control>
   <!-- Lidar (3D) -->
   <link name="lidar_link">
@@ -211,3 +272,30 @@
     </plugin>
   </gazebo>
+  <!-- Ground-truth world pose (Task 5 Step 3). This robot has no
+       OdometryPublisher (that was cavex_robot's wheeled/VelocityControl
+       approach) - a legged robot's true pose isn't a commanded-velocity
+       integral, so we publish the model's real simulator-internal pose
+       instead. Same honesty standard as cavex_robot's /odom: this is
+       simulator ground truth, not a claim about real-hardware sensing.
+       Bridged to ROS as geometry_msgs/PoseArray (gz.msgs.Pose_V) -
+       differs from cavex_robot's nav_msgs/Odometry-shaped ground truth, so
+       Task 10's ate_evaluator_node.py (which expects Odometry) needs a
+       small PoseArray -> Odometry republisher, not a direct bridge.
+       filename verified installed: `find / -iname "*pose-publisher*"` ->
+       libgz-sim8-pose-publisher-system.so / symlinked as
+       gz-sim-pose-publisher-system.so; class name gz::sim::systems::
+       PosePublisher confirmed via `strings` on that .so. -->
+  <gazebo>
+    <plugin filename="gz-sim-pose-publisher-system" name="gz::sim::systems::PosePublisher">
+      <publish_model_pose>true</publish_model_pose>
+      <publish_link_pose>false</publish_link_pose>
+      <publish_visual_pose>false</publish_visual_pose>
+      <publish_collision_pose>false</publish_collision_pose>
+      <publish_sensor_pose>false</publish_sensor_pose>
+      <publish_nested_model_pose>false</publish_nested_model_pose>
+      <use_pose_vector_msg>true</use_pose_vector_msg>
+      <static_publisher>false</static_publisher>
+      <update_frequency>30</update_frequency>
+    </plugin>
+  </gazebo>
 </robot>
