Commit message: Task 7 fix round 1 (cont.): add foot collision geometry
Hypothesis: the empty foot_link (no <collision>, only the shank
cylinder above it touches ground) gives the gait no real contact
point to push off from. Added a small sphere collision + higher ODE
surface friction (mu1/mu2=1.5) at each foot.

Tested clean (single, verified-non-duplicated Gazebo/ROS2 process
tree — an earlier test round was contaminated by orphaned processes
from prior launches and gave unreliable readings). Result: still ~0
net body translation under a real 15s forward /cmd_vel command.

Deeper root cause found instead: measured /joint_states never
approaches the commanded /joint_group_position_controller/joint_trajectory
setpoints at all (e.g. thigh commanded ~0.3-0.6 rad, measured stays
~0.015 rad) despite position_proportional_gain=300, active controllers,
and correctly-flowing trajectory messages (single-point streaming,
time_from_start~17ms, matches champ's 200Hz gait loop). This points at
JointTrajectoryController/gz_ros2_control not actually converging to
commanded positions in the sim loop -- a deeper ros2_control tuning or
integration issue this fix round did not resolve. Keeping the foot
collision (still a legitimate, independently-correct fix) but the
walker still cannot be shown to walk.

File: ros2_ws/src/cavex_slam_nav/urdf/cavex_walker.urdf.xacro (robot description, xacro)
@@ -145,9 +145,30 @@
     </joint>
     <!-- Virtual foot frame: fixed, offset by -shank_length from the knee.
-         Not a controlled joint (see header comment) - exists solely so
-         champ's links_map has a real 4th link per leg with the correct
-         shank length baked into its FK, matching quadruped_leg.h's
-         hip/upper_leg/lower_leg/foot 4-element joint_chain. -->
-    <link name="${prefix}_foot_link"/>
+         Originally exists solely so champ's links_map has a real 4th link
+         per leg with the correct shank length baked into its FK (see
+         header comment) - but an empty link with no <collision> means the
+         only ground-contact surface on the whole leg is the shank cylinder
+         well above the foot, which barely grazes the floor during the
+         gait's stance/swing cycle. Found empirically (Task 7 fix round 1):
+         with stance now held correctly (position_proportional_gain fix),
+         the walker still produced ~0 net displacement under a real forward
+         /cmd_vel - the legs cycle through the correct commanded gait angles
+         but generate no measurable push-off. Adding a real small-sphere
+         collision here, plus higher ODE surface friction than the default
+         (~1.0), gives the gait a real contact point to plant and push
+         against. -->
+    <link name="${prefix}_foot_link">
+      <visual>
+        <geometry><sphere radius="0.04"/></geometry>
+        <material name="black"><color rgba="0 0 0 1"/></material>
+      </visual>
+      <collision>
+        <geometry><sphere radius="0.04"/></geometry>
+      </collision>
+      <inertial>
+        <mass value="0.1"/>
+        <inertia ixx="0.0001" ixy="0" ixz="0" iyy="0.0001" iyz="0" izz="0.0001"/>
+      </inertial>
+    </link>
     <joint name="${prefix}_foot_joint" type="fixed">
       <parent link="${prefix}_knee_link"/>
@@ -155,4 +176,8 @@
       <origin xyz="0 0 -${shank_length}" rpy="0 0 0"/>
     </joint>
+    <gazebo reference="${prefix}_foot_link">
+      <mu1>1.5</mu1>
+      <mu2>1.5</mu2>
+    </gazebo>
   </xacro:macro>
   <xacro:champ_leg prefix="lf" x_sign="1"  y_sign="1"/>
